Commit message: update urdf file

File: description/robot.urdf.xacro (robot description, xacro)
@@ -2,4 +2,4 @@
 <robot xmlns:xacro="http://www.ros.org/wiki/xacro"  name="robot">
     <xacro:include filename="robot_core.xacro" />
-    <xacro:include filename="gazebo_control.xacro"/>
+    <xacro:include filename="gazebo_parameters.xacro"/>
 </robot>

File: description/robot_core.xacro (robot description, xacro)
@@ -1,150 +1,281 @@
 <?xml version="1.0"?>
-<robot xmlns:xacro="http://www.ros.org/wiki/xacro"  >
-    <xacro:include filename="inertial_macros.xacro"/>
-    <material name="white">
-        <color rgba="1 1 1 1" />
-    </material>
-    <material name="orange">
-        <color rgba="1 0.3 0.1 1" />
-    </material>
-    <material name="blue">
-        <color rgba="0.2 0.2 1 1" />
-    </material>
-    <material name="black">
-        <color rgba="0 0 0 1" />
-    </material>
-    <!-- BASE LINK -->
+<!-- This is the main structure of the robot. it has links, joints and material properties-->
+<robot xmlns:xacro="http://ros.org/wiki/xacro">
+  <!--xacro:property name="pi" value="3.14159" /-->
+  <xacro:include filename="materials.xacro" />
+  <xacro:include filename="robot_physical_properties.xacro" />
+  <xacro:include filename="inertial_macros.xacro" />
+    <link name="base_footprint">
+    </link>
+    <!-- chassis link of the robot -->
+    <joint name="base_joint" type="fixed">
+        <parent link="base_footprint" />
+        <child link="base_link" />
+        <origin xyz="0 0 ${base_height/2+wheel_radius/2}" rpy="0 0 0" />
+    </joint>
     <link name="base_link">
-    </link>
-    <!-- CHASSIS LINK-->
-    <joint name="chassis_joint" type="fixed">
-        <parent link="base_link"/>
-        <child link="chassis"/>
-        <origin xyz="-0.21 0 0"/>
-    </joint>
-    <link name="chassis">
         <visual>
-            <origin xyz="0.21 0 0.065"/>
+            <origin xyz="0 0 0" rpy="0 0 0"/>
             <geometry>
-                <box size="0.42 0.17 0.13"/>
+                <box size="${base_length} ${base_width} ${base_height}" />
             </geometry>
             <material name="white"/>
         </visual>
         <collision>
-            <origin xyz="0.21 0 0.065"/>
+            <origin xyz="0 0 0" rpy="0 0 0"/>
             <geometry>
-                <box size="0.42 0.17 0.13"/>
+                <box size="${base_length} ${base_width} ${base_height}" />
             </geometry>
         </collision>
-        <xacro:inertial_box mass="0.75" x="0.42" y="0.17" z="0.13">
-            <origin xyz="0.21 0 0.065" rpy="0 0 0"/>
+        <xacro:inertial_box mass="${base_mass}" x="${base_length}" y="${base_width}" z="${base_height}">
+            <origin xyz="0 0 0" rpy="0 0 0"/>
         </xacro:inertial_box>
     </link>
-    <gazebo reference="chassis">
-        <material>Gazebo/White</material>
-    </gazebo>
-    <!-- REAR LEFT WHEEL -->
-    <joint name="rear_left_wheel_joint" type="continuous">
-        <parent link="base_link"/>
-        <child link="rear_left_wheel"/>
-        <origin xyz="-0.16 0.1075 0" rpy="-${pi/2} 0 0"/>
-        <axis xyz="0 0 1"/>
-    </joint>
-    <link name="rear_left_wheel">
+    <link name="front_left_wheel_connector">
         <visual>
+            <origin xyz="0 0 0" rpy="0 0 0" />
             <geometry>
-                <cylinder length="0.045" radius="0.05" />
+                <cylinder radius="${wheel_connector_radius}" length="${wheel_connector_length}" />
             </geometry>
-            <material name="black"/>
+            <material name="red"/>
         </visual>
-        <collision>
-            <geometry>
-                <cylinder length="0.045" radius="0.05" />
-            </geometry>
-        </collision>
-        <xacro:inertial_cylinder mass="0.1" length="0.045" radius="0.05">
-            <origin xyz="0 0 0" rpy="0 0 0"/>
-        </xacro:inertial_cylinder>
-    </link>
-    <gazebo reference="rear_left_wheel">
-        <material>Gazebo/Black</material>
-    </gazebo>
-    <!-- REAR RIGHT WHEEL -->
-    <joint name="rear_right_wheel_joint" type="continuous">
-        <parent link="base_link"/>
-        <child link="rear_right_wheel"/>
-        <origin xyz="-0.16 -0.1075 0" rpy="${pi/2} 0 0"/>
-        <axis xyz="0 0 -1"/>
-    </joint>
-    <link name="rear_right_wheel">
-        <visual>
-            <geometry>
-                <cylinder length="0.045" radius="0.05" />
-            </geometry>
-            <material name="black"/>
-        </visual>
-        <collision>
-            <geometry>
-                <cylinder length="0.045" radius="0.05" />
-            </geometry>
-        </collision>
-        <xacro:inertial_cylinder mass="0.1" length="0.045" radius="0.05">
-            <origin xyz="0 0 0" rpy="0 0 0"/>
-        </xacro:inertial_cylinder>
-    </link>
-    <gazebo reference="rear_right_wheel">
-        <material>Gazebo/Black</material>
-    </gazebo>
-        <!-- FRONT LEFT WHEEL -->
-    <joint name="front_left_wheel_joint" type="continuous">
-        <parent link="base_link"/>
-        <child link="front_left_wheel"/>
-        <origin xyz="0.16 0.1075 0" rpy="-${pi/2} 0 0"/>
-        <axis xyz="0 0 1"/>
-    </joint>
-    <link name="front_left_wheel">
-        <visual>
-            <geometry>
-                <cylinder length="0.045" radius="0.05" />
-            </geometry>
-            <material name="black"/>
-        </visual>
-        <collision>
-            <geometry>
-                <cylinder length="0.045" radius="0.05" />
-            </geometry>
-        </collision>
-        <xacro:inertial_cylinder mass="0.1" length="0.045" radius="0.05">
-            <origin xyz="0 0 0" rpy="0 0 0"/>
-        </xacro:inertial_cylinder>
-    </link>
-    <gazebo reference="front_left_wheel">
-        <material>Gazebo/Black</material>
-    </gazebo>
-    <!-- FRONT RIGHT WHEEL -->
-    <joint name="front_right_wheel_joint" type="continuous">
-        <parent link="base_link"/>
-        <child link="front_right_wheel"/>
-        <origin xyz="0.16 -0.1075 0" rpy="${pi/2} 0 0"/>
-        <axis xyz="0 0 -1"/>
-    </joint>
-    <link name="front_right_wheel">
-        <visual>
-            <geometry>
-                <cylinder length="0.045" radius="0.05" />
-            </geometry>
-            <material name="black"/>
-        </visual>
-        <collision>
-            <geometry>
-                <cylinder length="0.045" radius="0.05" />
-            </geometry>
-        </collision>
-        <xacro:inertial_cylinder mass="0.1" length="0.045" radius="0.05">
-            <origin xyz="0 0 0" rpy="0 0 0"/>
-        </xacro:inertial_cylinder>
-    </link>
-    <gazebo reference="front_right_wheel">
-        <material>Gazebo/Black</material>
-    </gazebo>
+    <collision>
+      <origin xyz="0 0 0" rpy="0 0 0" />
+      <geometry>
+        <cylinder radius="${wheel_connector_radius}" length="${wheel_connector_length}" />
+      </geometry>
+    </collision>
+    <xacro:inertial_cylinder mass="${wheel_connector_mass}" length="${wheel_connector_length}" radius="${wheel_connector_radius}">
+      <origin xyz="0 0 0" rpy="0 0 0"/>
+    </xacro:inertial_cylinder>
+  </link>
+  <link name="front_right_wheel_connector">
+    <visual>
+      <origin xyz="0 0 0" rpy="0 0 0" />
+      <geometry>
+        <cylinder radius="${wheel_connector_radius}" length="${wheel_connector_length}" />
+      </geometry>
+      <material name="red"/>
+    </visual>
+    <collision>
+      <origin xyz="0 0 0" rpy="0 0 0" />
+      <geometry>
+        <cylinder radius="${wheel_connector_radius}" length="${wheel_connector_length}" />
+      </geometry>
+    </collision>
+    <xacro:inertial_cylinder mass="${wheel_connector_mass}" length="${wheel_connector_length}" radius="${wheel_connector_radius}">
+      <origin xyz="0 0 0" rpy="0 0 0"/>
+    </xacro:inertial_cylinder>
+  </link>
+  <link name="rear_left_wheel_connector">
+    <visual>
+      <origin xyz="0 0 0" rpy="0 0 0" />
+      <geometry>
+        <cylinder radius="${wheel_connector_radius}" length="${wheel_connector_length}" />
+      </geometry>
+      <material name="red"/>
+    </visual>
+    <collision>
+      <origin xyz="0 0 0" rpy="0 0 0" />
+      <geometry>
+        <cylinder radius="${wheel_connector_radius}" length="${wheel_connector_length}" />
+      </geometry>
+    </collision>
+    <xacro:inertial_cylinder mass="${wheel_connector_mass}" length="${wheel_connector_length}" radius="${wheel_connector_radius}">
+      <origin xyz="0 0 0" rpy="0 0 0"/>
+    </xacro:inertial_cylinder>
+  </link>
+  <link name="rear_right_wheel_connector">
+    <visual>
+      <origin xyz="0 0 0" rpy="0 0 0" />
+      <geometry>
+        <cylinder radius="${wheel_connector_radius}" length="${wheel_connector_length}" />
+      </geometry>
+      <material name="red"/>
+    </visual>
+    <collision>
+      <origin xyz="0 0 0" rpy="0 0 0" />
+      <geometry>
+        <cylinder radius="${wheel_connector_radius}" length="${wheel_connector_length}" />
+      </geometry>
+    </collision>
+    <xacro:inertial_cylinder mass="${wheel_connector_mass}" length="${wheel_connector_length}" radius="${wheel_connector_radius}">
+      <origin xyz="0 0 0" rpy="0 0 0"/>
+    </xacro:inertial_cylinder>
+  </link>
+<!-- Front left wheel -->
+  <link name="front_left_wheel_link">
+    <visual>
+      <origin xyz="0 0 0" rpy="0 0 0"/>
+      <geometry>
+        <cylinder radius="${wheel_radius}" length="${wheel_length}" />
+      </geometry>
+      <material name="black"/>
+    </visual>
+    <collision>
+      <origin xyz="0 0 0" rpy="0 0 0"/>
+      <geometry>
+        <cylinder radius="${wheel_radius}" length="${wheel_length}" />
+      </geometry>
+    </collision>
+    <xacro:inertial_cylinder mass="${wheel_mass}" length="${wheel_length}" radius="${wheel_radius}">
+      <origin xyz="0 0 0" rpy="0 0 0"/>
+    </xacro:inertial_cylinder>
+  </link>
+  <!-- Front left wheel steering -->
+  <link name="front_left_steering_link">
+    <visual>
+      <origin xyz="0 0 0" rpy="0 0 0" />
+      <geometry>
+        <cylinder radius="0.001" length="0.01" />
+      </geometry>
+    </visual>
+    <collision>
+      <origin xyz="0 0 0" rpy="0 0 0" />
+      <geometry>
+        <cylinder radius="0.001" length="0.01" />
+      </geometry>
+    </collision>
+    <xacro:inertial_cylinder mass="0.001" length="0.001" radius="0.01">
+      <origin xyz="0 0 0" rpy="0 0 0"/>
+    </xacro:inertial_cylinder>
+  </link>
+  <!-- Front right wheel -->
+  <link name="front_right_wheel_link">
+    <visual>
+      <origin xyz="0 0 0" rpy="0 0 0"/>
+      <geometry>
+        <cylinder radius="${wheel_radius}" length="${wheel_length}" />
+      </geometry>
+      <material name="black"/>
+    </visual>
+    <collision>
+      <origin xyz="0 0 0" rpy="0 0 0"/>
+      <geometry>
+        <cylinder radius="${wheel_radius}" length="${wheel_length}" />
+      </geometry>
+    </collision>
+    <xacro:inertial_cylinder mass="${wheel_mass}" length="${wheel_length}" radius="${wheel_radius}">
+      <origin xyz="0 0 0" rpy="0 0 0"/>
+    </xacro:inertial_cylinder>
+  </link>
+  <!-- Front right wheel steering -->
+  <link name="front_right_steering_link">
+    <visual>
+      <origin xyz="0 0 0" rpy="0 0 0" />
+      <geometry>
+        <cylinder radius="0.001" length="0.01" />
+      </geometry>
+    </visual>
+    <collision>
+      <origin xyz="0 0 0" rpy="0 0 0" />
+      <geometry>
+        <cylinder radius="0.001" length="0.01" />
+      </geometry>
+    </collision>
+    <xacro:inertial_cylinder mass="0.001" length="0.001" radius="0.01">
+      <origin xyz="0 0 0" rpy="0 0 0"/>
+    </xacro:inertial_cylinder>
+  </link>
+  <!-- Rear Left Wheel-->
+  <link name="rear_left_wheel_link">
+    <visual>
+      <origin xyz="0 0 0" rpy="0 0 0"/>
+      <geometry>
+        <cylinder radius="${wheel_radius}" length="${wheel_length}" />
+      </geometry>
+      <material name="black"/>
+    </visual>
+    <collision>
+      <origin xyz="0 0 0" rpy="0 0 0"/>
+      <geometry>
+        <cylinder radius="${wheel_radius}" length="${wheel_length}" />
+      </geometry>
+    </collision>
+    <xacro:inertial_cylinder mass="${wheel_mass}" length="${wheel_length}" radius="${wheel_radius}">
+      <origin xyz="0 0 0" rpy="0 0 0"/>
+    </xacro:inertial_cylinder>
+  </link>
+  <!-- Rear right wheel -->
+  <link name="rear_right_wheel_link">
+    <visual>
+      <origin xyz="0 0 0" rpy="0 0 0"/>
+      <geometry>
+        <cylinder radius="${wheel_radius}" length="${wheel_length}" />
+      </geometry>
+      <material name="black"/>
+    </visual>
+    <collision>
+      <origin xyz="0 0 0" rpy="0 0 0"/>
+      <geometry>
+        <cylinder radius="${wheel_radius}" length="${wheel_length}" />
+      </geometry>
+    </collision>
+    <xacro:inertial_cylinder mass="${wheel_mass}" length="${wheel_length}" radius="${wheel_radius}">
+      <origin xyz="0 0 0" rpy="0 0 0"/>
+    </xacro:inertial_cylinder>
+  </link>
+  <!--Joints-->
+  <joint name="front_left_wheel_connector_joint" type="fixed">
+    <parent link="base_link" />
+    <child link="front_left_wheel_connector" />
+    <origin xyz="${base_length/2-0.05} ${base_width/2} -${wheel_radius-wheel_connector_radius}" rpy="-${3.1459/2} 0 0" />
+  </joint>
+  <joint name="front_left_steering_joint" type="revolute">
+    <parent link="front_left_wheel_connector" />
+    <child link="front_left_steering_link" />
+    <origin xyz="0 0 ${wheel_connector_length/2}" rpy="0 0 0" />
+    <axis xyz="0 1 0" />
+    <limit lower="-1.0" upper="1.0" effort="100" velocity="100" />
+  </joint>
+  <joint name="front_left_wheel_joint" type="continuous">
+    <parent link="front_left_steering_link" />
+    <child link="front_left_wheel_link" />
+    <origin xyz="0 0 0" rpy="0 0 0" />
+    <axis xyz="0 0 1" />
+    <limit effort="100" velocity="100" />
+  </joint>
+  <joint name="front_right_wheel_connector_joint" type="fixed">
+    <parent link="base_link" />
+    <child link="front_right_wheel_connector" />
+    <origin xyz="${base_length/2-0.05} -${base_width/2} -${wheel_radius-wheel_connector_radius}" rpy="-${3.1459/2} 0 0" />
+  </joint>
+  <joint name="front_right_steering_joint" type="revolute">
+    <parent link="front_right_wheel_connector" />
+    <child link="front_right_steering_link" />
+    <origin xyz="0 0 -${wheel_connector_length/2}" rpy="0 0 0" />
+    <axis xyz="0 1 0" />
+    <limit lower="-1.0" upper="1.0" effort="100" velocity="100" />
+  </joint>
+  <joint name="front_right_wheel_joint" type="continuous">
+    <parent link="front_right_steering_link" />
+    <child link="front_right_wheel_link" />
+    <origin xyz="0 0 0" rpy="0 0 0" />
+    <axis xyz="0 0 1" />
+    <limit effort="100" velocity="100" />
+  </joint>
+  <joint name="rear_left_wheel_connector_joint" type="fixed">
+    <parent link="base_link" />
+    <child link="rear_left_wheel_connector" />
+    <origin xyz="-${base_length/2-0.05} ${base_width/2} -${wheel_radius-wheel_connector_radius}" rpy="-${3.1459/2} 0 0" />
+  </joint>
+  <joint name="rear_right_wheel_connector_joint" type="fixed">
+    <parent link="base_link" />
+    <child link="rear_right_wheel_connector" />
+    <origin xyz="-${base_length/2-0.05} -${base_width/2} -${wheel_radius-wheel_connector_radius}" rpy="-${3.1459/2} 0 0" />
+  </joint>
+  <joint name="rear_left_wheel_joint" type="continuous">
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