Commit message: update controller

File: install/my_robot/share/my_robot/description/gazebo_parameters.xacro (robot description, xacro)
@@ -1 +1,54 @@
-/home/pawan/dev_ws/src/my_robot/description/gazebo_parameters.xacro
+<?xml version="1.0"?>
+<robot name="my_robot"
+  xmlns:xacro="http://ros.org/wiki/xacro">
+  <gazebo reference = "rear_right_wheel_link">
+    <mu1>10000000</mu1>
+    <mu2>10000000</mu2>
+    <!-- <kp>10000000</kp>
+    <kd>10000000</kd>
+    <minDepth>0.001</minDepth>
+    <maxVel>10</maxVel>
+    <fdir1>1 0 0</fdir1> -->
+  </gazebo>
+  <gazebo reference = "rear_left_wheel_link">
+    <mu1>10000000</mu1>
+    <mu2>10000000</mu2>
+    <!-- <kp>10000000</kp>
+    <kd>10000000</kd>
+    <minDepth>0.001</minDepth>
+    <maxVel>10</maxVel>
+    <fdir1>1 0 0</fdir1> -->
+  </gazebo>
+  <gazebo reference = "front_right_wheel_link">
+    <mu1>10000000</mu1>
+    <mu2>10000000</mu2>
+    <!-- <kp>10000000</kp>
+    <kd>10000000</kd>
+    <minDepth>0.001</minDepth>
+    <maxVel>10</maxVel>
+    <fdir1>1 0 0</fdir1> -->
+  </gazebo>
+  <gazebo reference = "front_left_wheel_link">
+    <mu1>10000000</mu1>
+    <mu2>10000000</mu2>
+    <!-- <kp>10000000</kp>
+    <kd>10000000</kd>
+    <minDepth>0.001</minDepth>
+    <maxVel>10</maxVel>
+    <fdir1>1 0 0</fdir1> -->
+  </gazebo>
+  <gazebo>
+    <plugin filename ="gz_ros2_control-system" name = "gz_ros2_control::GazeboSimROS2ControlPlugin">
+      <parameters>$(find my_robot)/config/controllers.yaml</parameters>
+    </plugin>
+    <plugin filename="gz-sim-joint-state-publisher-system" name="gz::sim::systems::JointStatePublisher">
+      <topic>joint_states</topic>
+      <joint_name>front_left_steering_joint</joint_name>
+      <joint_name>front_right_steering_joint</joint_name>
+      <joint_name>front_left_wheel_joint</joint_name>
+      <joint_name>front_right_wheel_joint</joint_name>
+      <joint_name>rear_left_wheel_joint</joint_name>
+      <joint_name>rear_right_wheel_joint</joint_name>
+    </plugin>
+  </gazebo>
+</robot>

File: install/my_robot/share/my_robot/description/inertial_macros.xacro (robot description, xacro)
@@ -1 +1,23 @@
-/home/pawan/dev_ws/src/my_robot/description/inertial_macros.xacro
+<?xml version="1.0"?>
+<robot xmlns:xacro="http://www.ros.org/wiki/xacro" >
+    <!-- Specify some standard inertial calculations https://en.wikipedia.org/wiki/List_of_moments_of_inertia -->
+    <!-- These make use of xacro's mathematical functionality -->
+    <xacro:macro name="inertial_box" params="mass x y z *origin">
+        <inertial>
+            <xacro:insert_block name="origin"/>
+            <mass value="${mass}" />
+            <inertia ixx="${(1/12) * mass * (y*y+z*z)}" ixy="0.0" ixz="0.0"
+                    iyy="${(1/12) * mass * (x*x+z*z)}" iyz="0.0"
+                    izz="${(1/12) * mass * (x*x+y*y)}" />
+        </inertial>
+    </xacro:macro>
+    <xacro:macro name="inertial_cylinder" params="mass length radius *origin">
+        <inertial>
+            <xacro:insert_block name="origin"/>
+            <mass value="${mass}" />
+            <inertia ixx="${(1/12) * mass * (3*radius*radius + length*length)}" ixy="0.0" ixz="0.0"
+                    iyy="${(1/12) * mass * (3*radius*radius + length*length)}" iyz="0.0"
+                    izz="${(1/2) * mass * (radius*radius)}" />
+        </inertial>
+    </xacro:macro>
+</robot>

File: install/my_robot/share/my_robot/description/materials.xacro (robot description, xacro)
@@ -1 +1,21 @@
-/home/pawan/dev_ws/src/my_robot/description/materials.xacro
+<?xml version="1.0"?>
+<robot xmlns:xacro="http://ros.org/wiki/xacro">
+  <material name="black">
+    <color rgba=" 0 0 0 0.8" />
+  </material>
+  <material name="white">
+    <color rgba=" 1 1 1 0.8" />
+  </material>
+  <material name="red">
+    <color rgba=" 1 0 0 1" />
+  </material>
+  <material name="green">
+    <color rgba=" 0 1 0 1" />
+  </material>
+  <material name="blue">
+    <color rgba=" 0 0 1 1" />
+  </material>
+  <material name="grey">
+    <color rgba="0.25 0.25 0.25 1.0" />
+  </material>
+</robot>

File: install/my_robot/share/my_robot/description/odom_plugin.xacro (robot description, xacro)
@@ -1 +1,16 @@
-/home/pawan/dev_ws/src/my_robot/description/odom_plugin.xacro
+<?xml version="1.0"?>
+<robot xmlns:xacro="http://ros.org/wiki/xacro">
+  <!-- Gazebo odometry plugin -->
+  <gazebo>
+    <plugin filename="ignition-gazebo-odometry-publisher-system"
+            name="ignition::gazebo::systems::OdometryPublisher">
+      <robot_base_frame>base_footprint</robot_base_frame>
+      <odom_frame>odom</odom_frame>
+      <odom_topic>odom</odom_topic>
+      <tf_topic>tf</tf_topic>
+      <odom_publish_frequency>50.0</odom_publish_frequency>
+      <publish_tf>true</publish_tf>
+      <gaussian_noise>0.01</gaussian_noise>
+    </plugin>
+  </gazebo>
+</robot>

File: install/my_robot/share/my_robot/description/robot.urdf.xacro (robot description, xacro)
@@ -1 +1,8 @@
-/home/pawan/dev_ws/src/my_robot/description/robot.urdf.xacro
+<?xml version="1.0"?>
+<robot xmlns:xacro="http://www.ros.org/wiki/xacro"  name="robot">
+    <xacro:include filename="robot_core.xacro" />
+    <xacro:include filename="gazebo_parameters.xacro"/>
+    <xacro:include filename="ros2_control.xacro" />
+    <xacro:include filename="transmission.xacro" />
+    <xacro:include filename="odom_plugin.xacro" />
+</robot>

File: install/my_robot/share/my_robot/description/robot_core.xacro (robot description, xacro)
@@ -1 +1,281 @@
-/home/pawan/dev_ws/src/my_robot/description/robot_core.xacro
+<?xml version="1.0"?>
+<!-- This is the main structure of the robot. it has links, joints and material properties-->
+<robot xmlns:xacro="http://ros.org/wiki/xacro">
+  <!--xacro:property name="pi" value="3.14159" /-->
+  <xacro:include filename="materials.xacro" />
+  <xacro:include filename="robot_physical_properties.xacro" />
+  <xacro:include filename="inertial_macros.xacro" />
+    <link name="base_footprint">
+    </link>
+    <!-- chassis link of the robot -->
+    <joint name="base_joint" type="fixed">
+        <parent link="base_footprint" />
+        <child link="base_link" />
+        <origin xyz="0 0 ${base_height/2+wheel_radius/2}" rpy="0 0 0" />
+    </joint>
+    <link name="base_link">
+        <visual>
+            <origin xyz="0 0 0" rpy="0 0 0"/>
+            <geometry>
+                <box size="${base_length} ${base_width} ${base_height}" />
+            </geometry>
+            <material name="white"/>
+        </visual>
+        <collision>
+            <origin xyz="0 0 0" rpy="0 0 0"/>
+            <geometry>
+                <box size="${base_length} ${base_width} ${base_height}" />
+            </geometry>
+        </collision>
+        <xacro:inertial_box mass="${base_mass}" x="${base_length}" y="${base_width}" z="${base_height}">
+            <origin xyz="0 0 0" rpy="0 0 0"/>
+        </xacro:inertial_box>
+    </link>
+    <link name="front_left_wheel_connector">
+        <visual>
+            <origin xyz="0 0 0" rpy="0 0 0" />
+            <geometry>
+                <cylinder radius="${wheel_connector_radius}" length="${wheel_connector_length}" />
+            </geometry>
+            <material name="red"/>
+        </visual>
+    <collision>
+      <origin xyz="0 0 0" rpy="0 0 0" />
+      <geometry>
+        <cylinder radius="${wheel_connector_radius}" length="${wheel_connector_length}" />
+      </geometry>
+    </collision>
+    <xacro:inertial_cylinder mass="${wheel_connector_mass}" length="${wheel_connector_length}" radius="${wheel_connector_radius}">
+      <origin xyz="0 0 0" rpy="0 0 0"/>
+    </xacro:inertial_cylinder>
+  </link>
+  <link name="front_right_wheel_connector">
+    <visual>
+      <origin xyz="0 0 0" rpy="0 0 0" />
+      <geometry>
+        <cylinder radius="${wheel_connector_radius}" length="${wheel_connector_length}" />
+      </geometry>
+      <material name="red"/>
+    </visual>
+    <collision>
+      <origin xyz="0 0 0" rpy="0 0 0" />
+      <geometry>
+        <cylinder radius="${wheel_connector_radius}" length="${wheel_connector_length}" />
+      </geometry>
+    </collision>
+    <xacro:inertial_cylinder mass="${wheel_connector_mass}" length="${wheel_connector_length}" radius="${wheel_connector_radius}">
+      <origin xyz="0 0 0" rpy="0 0 0"/>
+    </xacro:inertial_cylinder>
+  </link>
+  <link name="rear_left_wheel_connector">
+    <visual>
+      <origin xyz="0 0 0" rpy="0 0 0" />
+      <geometry>
+        <cylinder radius="${wheel_connector_radius}" length="${wheel_connector_length}" />
+      </geometry>
+      <material name="red"/>
+    </visual>
+    <collision>
+      <origin xyz="0 0 0" rpy="0 0 0" />
+      <geometry>
+        <cylinder radius="${wheel_connector_radius}" length="${wheel_connector_length}" />
+      </geometry>
+    </collision>
+    <xacro:inertial_cylinder mass="${wheel_connector_mass}" length="${wheel_connector_length}" radius="${wheel_connector_radius}">
+      <origin xyz="0 0 0" rpy="0 0 0"/>
+    </xacro:inertial_cylinder>
+  </link>
+  <link name="rear_right_wheel_connector">
+    <visual>
+      <origin xyz="0 0 0" rpy="0 0 0" />
+      <geometry>
+        <cylinder radius="${wheel_connector_radius}" length="${wheel_connector_length}" />
+      </geometry>
+      <material name="red"/>
+    </visual>
+    <collision>
+      <origin xyz="0 0 0" rpy="0 0 0" />
+      <geometry>
+        <cylinder radius="${wheel_connector_radius}" length="${wheel_connector_length}" />
+      </geometry>
+    </collision>
+    <xacro:inertial_cylinder mass="${wheel_connector_mass}" length="${wheel_connector_length}" radius="${wheel_connector_radius}">
+      <origin xyz="0 0 0" rpy="0 0 0"/>
+    </xacro:inertial_cylinder>
+  </link>
+<!-- Front left wheel -->
+  <link name="front_left_wheel_link">
+    <visual>
+      <origin xyz="0 0 0" rpy="0 0 0"/>
+      <geometry>
+        <cylinder radius="${wheel_radius}" length="${wheel_length}" />
+      </geometry>
+      <material name="black"/>
+    </visual>
+    <collision>
+      <origin xyz="0 0 0" rpy="0 0 0"/>
+      <geometry>
+        <cylinder radius="${wheel_radius}" length="${wheel_length}" />
+      </geometry>
+    </collision>
+    <xacro:inertial_cylinder mass="${wheel_mass}" length="${wheel_length}" radius="${wheel_radius}">
+      <origin xyz="0 0 0" rpy="0 0 0"/>
+    </xacro:inertial_cylinder>
+  </link>
+  <!-- Front left wheel steering -->
+  <link name="front_left_steering_link">
+    <visual>
+      <origin xyz="0 0 0" rpy="0 0 0" />
+      <geometry>
+        <cylinder radius="0.001" length="0.01" />
+      </geometry>
+    </visual>
+    <collision>
+      <origin xyz="0 0 0" rpy="0 0 0" />
+      <geometry>
+        <cylinder radius="0.001" length="0.01" />
+      </geometry>
+    </collision>
+    <xacro:inertial_cylinder mass="0.001" length="0.001" radius="0.01">
+      <origin xyz="0 0 0" rpy="0 0 0"/>
+    </xacro:inertial_cylinder>
+  </link>
+  <!-- Front right wheel -->
+  <link name="front_right_wheel_link">
+    <visual>
+      <origin xyz="0 0 0" rpy="0 0 0"/>
+      <geometry>
+        <cylinder radius="${wheel_radius}" length="${wheel_length}" />
+      </geometry>
+      <material name="black"/>
+    </visual>
+    <collision>
+      <origin xyz="0 0 0" rpy="0 0 0"/>
+      <geometry>
+        <cylinder radius="${wheel_radius}" length="${wheel_length}" />
+      </geometry>
+    </collision>
+    <xacro:inertial_cylinder mass="${wheel_mass}" length="${wheel_length}" radius="${wheel_radius}">
+      <origin xyz="0 0 0" rpy="0 0 0"/>
+    </xacro:inertial_cylinder>
+  </link>
+  <!-- Front right wheel steering -->
+  <link name="front_right_steering_link">
+    <visual>
+      <origin xyz="0 0 0" rpy="0 0 0" />
+      <geometry>
+        <cylinder radius="0.001" length="0.01" />
+      </geometry>
+    </visual>
+    <collision>
+      <origin xyz="0 0 0" rpy="0 0 0" />
+      <geometry>
+        <cylinder radius="0.001" length="0.01" />
+      </geometry>
+    </collision>
+    <xacro:inertial_cylinder mass="0.001" length="0.001" radius="0.01">
+      <origin xyz="0 0 0" rpy="0 0 0"/>
+    </xacro:inertial_cylinder>
+  </link>
+  <!-- Rear Left Wheel-->
+  <link name="rear_left_wheel_link">
+    <visual>
+      <origin xyz="0 0 0" rpy="0 0 0"/>
+      <geometry>
+        <cylinder radius="${wheel_radius}" length="${wheel_length}" />
+      </geometry>
+      <material name="black"/>
+    </visual>
+    <collision>
+      <origin xyz="0 0 0" rpy="0 0 0"/>
+      <geometry>
+        <cylinder radius="${wheel_radius}" length="${wheel_length}" />
+      </geometry>
+    </collision>
+    <xacro:inertial_cylinder mass="${wheel_mass}" length="${wheel_length}" radius="${wheel_radius}">
+      <origin xyz="0 0 0" rpy="0 0 0"/>
+    </xacro:inertial_cylinder>
+  </link>
+  <!-- Rear right wheel -->
+  <link name="rear_right_wheel_link">
+    <visual>
+      <origin xyz="0 0 0" rpy="0 0 0"/>
+      <geometry>
+        <cylinder radius="${wheel_radius}" length="${wheel_length}" />
+      </geometry>
+      <material name="black"/>
+    </visual>
+    <collision>
+      <origin xyz="0 0 0" rpy="0 0 0"/>
+      <geometry>
+        <cylinder radius="${wheel_radius}" length="${wheel_length}" />
+      </geometry>
+    </collision>
+    <xacro:inertial_cylinder mass="${wheel_mass}" length="${wheel_length}" radius="${wheel_radius}">
+      <origin xyz="0 0 0" rpy="0 0 0"/>
+    </xacro:inertial_cylinder>
+  </link>
+  <!--Joints-->
+  <joint name="front_left_wheel_connector_joint" type="fixed">
+    <parent link="base_link" />
+    <child link="front_left_wheel_connector" />
+    <origin xyz="${base_length/2-0.05} ${base_width/2} -${wheel_radius-wheel_connector_radius}" rpy="-${3.1459/2} 0 0" />
+  </joint>
+  <joint name="front_left_steering_joint" type="revolute">
+    <parent link="front_left_wheel_connector" />
+    <child link="front_left_steering_link" />
+    <origin xyz="0 0 ${wheel_connector_length/2}" rpy="0 0 0" />
+    <axis xyz="0 1 0" />
+    <limit lower="-1.0" upper="1.0" effort="100" velocity="100" />
+  </joint>
+  <joint name="front_left_wheel_joint" type="continuous">
+    <parent link="front_left_steering_link" />
+    <child link="front_left_wheel_link" />
+    <origin xyz="0 0 0" rpy="0 0 0" />
+    <axis xyz="0 0 1" />
+    <limit effort="100" velocity="100" />
+  </joint>
+  <joint name="front_right_wheel_connector_joint" type="fixed">
+    <parent link="base_link" />
+    <child link="front_right_wheel_connector" />
+    <origin xyz="${base_length/2-0.05} -${base_width/2} -${wheel_radius-wheel_connector_radius}" rpy="-${3.1459/2} 0 0" />
+  </joint>
+  <joint name="front_right_steering_joint" type="revolute">
+    <parent link="front_right_wheel_connector" />
+    <child link="front_right_steering_link" />
+    <origin xyz="0 0 -${wheel_connector_length/2}" rpy="0 0 0" />
+    <axis xyz="0 1 0" />
+    <limit lower="-1.0" upper="1.0" effort="100" velocity="100" />
+  </joint>
+  <joint name="front_right_wheel_joint" type="continuous">
+    <parent link="front_right_steering_link" />
+    <child link="front_right_wheel_link" />
+    <origin xyz="0 0 0" rpy="0 0 0" />
+    <axis xyz="0 0 1" />
+    <limit effort="100" velocity="100" />
+  </joint>
+  <joint name="rear_left_wheel_connector_joint" type="fixed">
+    <parent link="base_link" />
+    <child link="rear_left_wheel_connector" />
+    <origin xyz="-${base_length/2-0.05} ${base_width/2} -${wheel_radius-wheel_connector_radius}" rpy="-${3.1459/2} 0 0" />
+  </joint>
+  <joint name="rear_right_wheel_connector_joint" type="fixed">
+    <parent link="base_link" />
+    <child link="rear_right_wheel_connector" />
+    <origin xyz="-${base_length/2-0.05} -${base_width/2} -${wheel_radius-wheel_connector_radius}" rpy="-${3.1459/2} 0 0" />
+  </joint>
+  <joint name="rear_left_wheel_joint" type="continuous">
+    <parent link="rear_left_wheel_connector" />
+    <child link="rear_left_wheel_link" />
+    <origin xyz="0 0 ${wheel_connector_length/2}" rpy="0 0 0" />
+    <axis xyz="0 0 1" />
+    <limit effort="100" velocity="100" />
+  </joint>
+  <joint name="rear_right_wheel_joint" type="continuous">
+    <parent link="rear_right_wheel_connector" />
+    <child link="rear_right_wheel_link" />
+    <origin xyz="0 0 -${wheel_connector_length/2}" rpy="0 0 0" />
+    <axis xyz="0 0 1" />
+    <limit effort="100" velocity="100" />
+  </joint>
+</robot>

File: install/my_robot/share/my_robot/description/robot_physical_properties.xacro (robot description, xacro)
@@ -1 +1,19 @@
-/home/pawan/dev_ws/src/my_robot/description/robot_physical_properties.xacro
+<?xml version="1.0"?>
+<robot xmlns:xacro="http://ros.org/wiki/xacro">
+    <!-- Constants for robot dimensions -->
+    <xacro:property name="base_mass" value="4.0" />
+    <xacro:property name="base_width" value="0.17" />
+    <xacro:property name="base_length" value="0.42" />
+    <xacro:property name="base_height" value="0.13" />
+    <xacro:property name="wheel_mass" value="0.3" />
+    <xacro:property name="wheel_length" value="0.045" />
+    <xacro:property name="wheel_radius" value="0.05" />
+    <xacro:property name="wheel_connector_length" value="0.1" />
+    <xacro:property name="wheel_connector_radius" value="0.01" />
+    <xacro:property name="wheel_connector_mass" value="0.01" />
+    <!--
+    <xacro:property name="bottom_to_top_connector_length" value="0.1" />
+    <xacro:property name="bottom_to_top_connector_radius" value="0.005" />
+    <xacro:property name="bottom_to_top_connector_mass" value="0.01"/>
+    -->
+</robot>

File: src/my_robot/description/odom_plugin.xacro (robot description, xacro)
@@ -1,13 +1,15 @@
 <?xml version="1.0"?>
-<robot name="my_robot"
-  xmlns:xacro="http://ros.org/wiki/xacro">
+<robot xmlns:xacro="http://ros.org/wiki/xacro">
+  <!-- Gazebo odometry plugin -->
   <gazebo>
-    <plugin filename='gz-sim-odometry-publisher-system' name='gz::sim::systems::OdometryPublisher' >
-      <dimensions>3</dimensions>
-      <odom_publish_frequency>50</odom_publish_frequency>
-      <odom_topic>/odom</odom_topic>
+    <plugin filename="ignition-gazebo-odometry-publisher-system"
+            name="ignition::gazebo::systems::OdometryPublisher">
+      <robot_base_frame>base_footprint</robot_base_frame>
       <odom_frame>odom</odom_frame>
-      <robot_base_frame>base_footprint</robot_base_frame>
-      <tf_topic>/tf</tf_topic>
+      <odom_topic>odom</odom_topic>
+      <tf_topic>tf</tf_topic>
+      <odom_publish_frequency>50.0</odom_publish_frequency>
+      <publish_tf>true</publish_tf>
+      <gaussian_noise>0.01</gaussian_noise>
     </plugin>
   </gazebo>

File: src/my_robot/description/robot.urdf.xacro (robot description, xacro)
@@ -3,3 +3,6 @@
     <xacro:include filename="robot_core.xacro" />
     <xacro:include filename="gazebo_parameters.xacro"/>
+    <xacro:include filename="ros2_control.xacro" />
+    <xacro:include filename="transmission.xacro" />
+    <xacro:include filename="odom_plugin.xacro" />
 </robot>
